Commit message: 加入tf，完成

File: src/rm_description/urdf/gimbal.urdf.xacro (robot description, xacro)
@@ -62,5 +62,5 @@
   <link name="shooter_link" />
   <joint name="shooter_joint" type="fixed">
-    <origin xyz="0.0032818 0 0.097945" rpy="0 0 0" />
+    <origin xyz="0.0032818 0 0.097945" rpy="${pi/2} 0 ${pi/2}" />
     <parent link="base_link" />
     <child link="shooter_link" />

Commit message: 修bug，关于tf

File: src/rm_description/urdf/gimbal.urdf.xacro (robot description, xacro)
@@ -62,5 +62,5 @@
   <link name="shooter_link" />
   <joint name="shooter_joint" type="fixed">
-    <origin xyz="0.0032818 0 0.097945" rpy="${pi/2} 0 ${pi/2}" />
+    <origin xyz="0.0032818 0 0.097945" rpy="0 0 0" />
     <parent link="base_link" />
     <child link="shooter_link" />
