Commit message: 修改英雄urdf文件

File: src/rm_description/urdf/gimbal_b3.urdf.xacro (robot description, xacro)
@@ -90,5 +90,5 @@
   </link>
   <joint name="camera_base_joint" type="fixed">
-    <origin xyz="0.06203 0.0 -0.04085" rpy="0 0 0" />
+    <origin xyz="0.06203 -0.05 0.17085" rpy="0 0 0" />
     <!-- <origin xyz="0.088 0.0 0.0585" rpy="0 0 0" /> -->
     <parent link="pitch_link" />
